Commit message: fixed path error

File: ezmile_ws/src/catvehicle/urdf/os1_64.urdf.xacro (robot description, xacro)
@@ -38,5 +38,5 @@
         <origin xyz="0 0 0" rpy="0 0 0"/>
         <geometry>
-          <mesh filename="package://ezmile_gen0/meshes/${file_visual}.stl" />
+          <mesh filename="package://catvehicle/meshes/${file_visual}.stl" />
         </geometry>
       </visual>
