Commit message: localization lidars committed

File: catkin_ws/src/4ws_robot/urdf/four_wheel_robot.xacro (robot description, xacro)
@@ -279,5 +279,5 @@
     </link>
     <!--Front Right Wheel-->
-    <joint name="front_right_wheel_joint" type="continuous">
+    <joint name="front_right_wheel_joint" type="fixed">
         <parent link="front_right_steering_link"/>
         <child link="front_right_wheel_link"/>
@@ -366,5 +366,5 @@
     </link>
 <!--Front Left Wheel-->
-    <joint name="front_left_wheel_joint" type="continuous">
+    <joint name="front_left_wheel_joint" type="fixed">
           <parent link="front_left_steering_link"/>
           <child link="front_left_wheel_link"/>
@@ -421,4 +421,9 @@
         </inertial>
     </link>
+<!-- Lidars to be installed -->
+  <xacro:include filename="$(find 4ws_robot)/urdf/os1_64.urdf.xacro"/>
+  <xacro:os1_64 parent="base" name="ouster" prefix="/os1_cloud_node" hz="20" samples="512">
+    <origin xyz="0 0 3.0" rpy="0 0 0" />
+  </xacro:os1_64>
 <!-- motors and transmissions for the two rear wheels -->
     <transmission name="tran1">
@@ -442,40 +447,40 @@
         </actuator>
     </transmission>
-    <transmission name="tran3">
+    <transmission name="steering_back_left_transmission">
         <type>transmission_interface/SimpleTransmission</type>
         <joint name="back_left_steering_joint">
             <hardwareInterface>hardware_interface/PositionJointInterface</hardwareInterface>
         </joint>
-        <actuator name="eps_b_left">
-            <hardwareInterface>hardware_interface/PositionJointInterface</hardwareInterface>
-            <mechanicalReduction>1</mechanicalReduction>
-        </actuator>
-    </transmission>
-        <transmission name="tran4">
+        <actuator name="steering_back_left_acutator">
+            <hardwareInterface>hardware_interface/PositionJointInterface</hardwareInterface>
+            <mechanicalReduction>1</mechanicalReduction>
+        </actuator>
+    </transmission>
+    <transmission name="steering_back_right_transmission">
         <type>transmission_interface/SimpleTransmission</type>
         <joint name="back_right_steering_joint">
             <hardwareInterface>hardware_interface/PositionJointInterface</hardwareInterface>
         </joint>
-        <actuator name="eps_b_right">
-            <hardwareInterface>hardware_interface/PositionJointInterface</hardwareInterface>
-            <mechanicalReduction>1</mechanicalReduction>
-        </actuator>
-    </transmission>
-    <transmission name="rack_and_pinion_left">
+        <actuator name="steering_back_right_acutator">
+            <hardwareInterface>hardware_interface/PositionJointInterface</hardwareInterface>
+            <mechanicalReduction>1</mechanicalReduction>
+        </actuator>
+    </transmission>
+    <transmission name="steering_front_left_transmission">
         <type>transmission_interface/SimpleTransmission</type>
         <joint name="front_left_steering_joint">
             <hardwareInterface>hardware_interface/PositionJointInterface</hardwareInterface>
         </joint>
-        <actuator name="eps_left">
-            <hardwareInterface>hardware_interface/PositionJointInterface</hardwareInterface>
-            <mechanicalReduction>1</mechanicalReduction>
-        </actuator>
-    </transmission>
-    <transmission name="rack_and_pinion_right">
+        <actuator name="steering_front_left_acutator">
+            <hardwareInterface>hardware_interface/PositionJointInterface</hardwareInterface>
+            <mechanicalReduction>1</mechanicalReduction>
+        </actuator>
+    </transmission>
+    <transmission name="steering_front_right_transmission">
         <type>transmission_interface/SimpleTransmission</type>
         <joint name="front_right_steering_joint">
             <hardwareInterface>hardware_interface/PositionJointInterface</hardwareInterface>
         </joint>
-        <actuator name="eps_right">
+        <actuator name="steering_front_right_acutator">
             <hardwareInterface>hardware_interface/PositionJointInterface</hardwareInterface>
             <mechanicalReduction>1</mechanicalReduction>

Commit message: cmd to gazebo

File: catkin_ws/src/4ws_robot/urdf/four_wheel_robot.xacro (robot description, xacro)
@@ -60,5 +60,5 @@
   <link name="base_link">
     <visual>
-      <origin xyz="0 0 0" rpy="0 0 1.57079633"/>
+      <origin xyz="0 0 0" rpy="0 0 -1.57079633"/>
       <geometry>
         <mesh filename="package://4ws_robot/meshes/gen0_colored.dae"/>
@@ -279,5 +279,5 @@
     </link>
     <!--Front Right Wheel-->
-    <joint name="front_right_wheel_joint" type="fixed">
+    <joint name="front_right_wheel_joint" type="continuous">
         <parent link="front_right_steering_link"/>
         <child link="front_right_wheel_link"/>
@@ -366,5 +366,5 @@
     </link>
 <!--Front Left Wheel-->
-    <joint name="front_left_wheel_joint" type="fixed">
+    <joint name="front_left_wheel_joint" type="continuous">
           <parent link="front_left_steering_link"/>
           <child link="front_left_wheel_link"/>
@@ -447,4 +447,24 @@
         </actuator>
     </transmission>
+    <!-- <transmission name="tran3">
+        <type>transmission_interface/SimpleTransmission</type>
+        <joint name="front_right_wheel_joint">
+            <hardwareInterface>hardware_interface/VelocityJointInterface</hardwareInterface>
+        </joint>
+        <actuator name="motor3">
+            <hardwareInterface>hardware_interface/VelocityJointInterface</hardwareInterface>
+            <mechanicalReduction>1</mechanicalReduction>
+        </actuator>
+    </transmission>
+    <transmission name="tran4">
+        <type>transmission_interface/SimpleTransmission</type>
+        <joint name="front_left_wheel_joint">
+            <hardwareInterface>hardware_interface/VelocityJointInterface</hardwareInterface>
+        </joint>
+        <actuator name="motor4">
+            <hardwareInterface>hardware_interface/VelocityJointInterface</hardwareInterface>
+            <mechanicalReduction>1</mechanicalReduction>
+        </actuator>
+    </transmission> -->
     <transmission name="steering_back_left_transmission">
         <type>transmission_interface/SimpleTransmission</type>

Commit message: Navigation stack

File: catkin_ws/src/4ws_robot/urdf/four_wheel_robot.xacro (robot description, xacro)
@@ -447,5 +447,5 @@
         </actuator>
     </transmission>
-    <!-- <transmission name="tran3">
+    <transmission name="tran3">
         <type>transmission_interface/SimpleTransmission</type>
         <joint name="front_right_wheel_joint">
@@ -466,5 +466,5 @@
             <mechanicalReduction>1</mechanicalReduction>
         </actuator>
-    </transmission> -->
+    </transmission>
     <transmission name="steering_back_left_transmission">
         <type>transmission_interface/SimpleTransmission</type>

File: catkin_ws/src/4ws_robot/urdf/os1_64.urdf.xacro (robot description, xacro)
@@ -3,5 +3,5 @@
 <robot xmlns:xacro="http://ros.org/wiki/xacro" name="os1_64">
   <xacro:property name="PI" value="3.1415926535897931"/>
-  <xacro:macro name="os1_64" params="*origin parent:=base name:=ouster reduced:=true prefix:=/os1_cloud_node hz:=10 samples:=512 min_range:=1.5 max_range:=100 noise:=0.008 min_angle_v:=-16.6 max_angle_v:=16.6 gpu:=true">
+  <xacro:macro name="os1_64" params="*origin parent:=base name:=ouster reduced:=true prefix:=/os1_cloud_node hz:=10 samples:=512 min_range:=1.5 max_range:=30 noise:=0.008 min_angle_v:=-16.6 max_angle_v:=16.6 gpu:=true">
     <!-- Conditional properties -->
     <xacro:if value="${reduced}">

Commit message: 4 lidars installed

File: catkin_ws/src/4ws_robot/urdf/four_wheel_robot.xacro (robot description, xacro)
@@ -423,7 +423,108 @@
 <!-- Lidars to be installed -->
   <xacro:include filename="$(find 4ws_robot)/urdf/os1_64.urdf.xacro"/>
-  <xacro:os1_64 parent="base" name="ouster" prefix="/os1_cloud_node" hz="20" samples="512">
+  <xacro:os1_64 parent="base" name="ouster" prefix="/os1_cloud_node" hz="10" samples="512">
     <origin xyz="0 0 3.0" rpy="0 0 0" />
   </xacro:os1_64>
+<!-- Lidars to be installed -->
+<joint name="sick_lidar_fl_joint" type="fixed">
+    <axis xyz="0 1 0" />
+    <origin xyz="1.9 0.8 0.3" rpy="${PI} 0 ${3*PI/4}"/>
+    <parent link="base_link"/>
+    <child link="sick_lidar_fl_link"/>
+  </joint>
+  <link name="sick_lidar_fl_link">
+    <collision>
+      <origin xyz="0 0 0" rpy="0 0 0"/>
+      <geometry>
+    <box size="0.1 0.1 0.1"/>
+      </geometry>
+    </collision>
+    <visual>
+      <origin xyz="0 0 0" rpy="0 0 0"/>
+      <geometry>
+        <mesh filename="package://4ws_robot/meshes/sick_lidar.obj"/>
+      </geometry>
+    </visual>
+    <inertial>
+      <mass value="1e-5" />
+      <origin xyz="0 0 0" rpy="0 0 0"/>
+      <inertia ixx="1e-6" ixy="0" ixz="0" iyy="1e-6" iyz="0" izz="1e-6" />
+    </inertial>
+  </link>
+<joint name="sick_lidar_fr_joint" type="fixed">
+    <axis xyz="0 1 0" />
+    <origin xyz="1.8 -0.8 0.3" rpy="${PI} 0 ${PI/4}"/>
+    <parent link="base_link"/>
+    <child link="sick_lidar_fr_link"/>
+  </joint>
+  <link name="sick_lidar_fr_link">
+    <collision>
+      <origin xyz="0 0 0" rpy="0 0 0"/>
+      <geometry>
+    <box size="0.1 0.1 0.1"/>
+      </geometry>
+    </collision>
+    <visual>
+      <origin xyz="0 0 0" rpy="0 0 0"/>
+      <geometry>
+        <mesh filename="package://4ws_robot/meshes/sick_lidar.obj"/>
+      </geometry>
+    </visual>
+    <inertial>
+      <mass value="1e-5" />
+      <origin xyz="0 0 0" rpy="0 0 0"/>
+      <inertia ixx="1e-6" ixy="0" ixz="0" iyy="1e-6" iyz="0" izz="1e-6" />
+    </inertial>
+  </link>
+  <joint name="sick_lidar_rl_joint" type="fixed">
+    <axis xyz="0 1 0" />
+    <origin xyz="-1.75 0.85 0.3" rpy="${PI} 0 ${5*PI/4}"/>
+    <parent link="base_link"/>
+    <child link="sick_lidar_rl_link"/>
+  </joint>
+  <link name="sick_lidar_rl_link">
+    <collision>
+      <origin xyz="0 0 0" rpy="0 0 0"/>
+      <geometry>
+    <box size="0.1 0.1 0.1"/>
+      </geometry>
+    </collision>
+    <visual>
+      <origin xyz="0 0 0" rpy="0 0 0"/>
+      <geometry>
+        <mesh filename="package://4ws_robot/meshes/sick_lidar.obj"/>
+      </geometry>
+    </visual>
+    <inertial>
+      <mass value="1e-5" />
+      <origin xyz="0 0 0" rpy="0 0 0"/>
+      <inertia ixx="1e-6" ixy="0" ixz="0" iyy="1e-6" iyz="0" izz="1e-6" />
+    </inertial>
+  </link>
+    <joint name="sick_lidar_rr_joint" type="fixed">
+    <axis xyz="0 1 0" />
+    <origin xyz="-1.85 -0.8 0.3" rpy="${PI} 0 ${-PI/4}"/>
+    <parent link="base_link"/>
+    <child link="sick_lidar_rr_link"/>
+  </joint>
+  <link name="sick_lidar_rr_link">
+    <collision>
+      <origin xyz="0 0 0" rpy="0 0 0"/>
+      <geometry>
+    <box size="0.1 0.1 0.1"/>
+      </geometry>
+    </collision>
+    <visual>
+      <origin xyz="0 0 0" rpy="0 0 0"/>
+      <geometry>
+        <mesh filename="package://4ws_robot/meshes/sick_lidar.obj"/>
+      </geometry>
+    </visual>
+    <inertial>
+      <mass value="1e-5" />
+      <origin xyz="0 0 0" rpy="0 0 0"/>
+      <inertia ixx="1e-6" ixy="0" ixz="0" iyy="1e-6" iyz="0" izz="1e-6" />
+    </inertial>
+  </link>
 <!-- motors and transmissions for the two rear wheels -->
     <transmission name="tran1">
@@ -513,3 +614,143 @@
   </plugin>
 </gazebo>
+<gazebo reference="sick_lidar_fl_link">
+    <sensor type="ray" name="sick_lidar_fl">
+      <pose>0 0 0 0 0 0</pose>
+      <visualize>true</visualize>
+      <update_rate>40</update_rate>
+      <ray>
+        <scan>
+          <horizontal>
+            <samples>720</samples>
+            <resolution>1</resolution>
+            <min_angle>0</min_angle>
+            <max_angle>3.141592</max_angle>
+          </horizontal>
+        </scan>
+        <range>
+          <min>0.5</min>
+          <max>30.0</max>
+          <resolution>0.01</resolution>
+        </range>
+        <noise>
+          <type>gaussian</type>
+          <!-- Noise parameters based on published spec for Hokuyo laser
+               achieving "+-30mm" accuracy at range < 10m.  A mean of 0.0m and
+               stddev of 0.01m will put 99.7% of samples within 0.03m of the true
+               reading. -->
+          <mean>0.0</mean>
+          <stddev>0.01</stddev>
+        </noise>
+      </ray>
+      <plugin name="gazebo_ros_fl_lidar" filename="libgazebo_ros_laser.so">
+        <topicName>sick_lidar_fl/scan</topicName>
+        <frameName>sick_lidar_fl_link</frameName>
+      </plugin>
+    </sensor>
+  </gazebo>
+<gazebo reference="sick_lidar_fr_link">
+    <sensor type="ray" name="sick_lidar_fr">
+      <pose>0 0 0 0 0 0</pose>
+      <visualize>true</visualize>
+      <update_rate>40</update_rate>
+      <ray>
+        <scan>
+          <horizontal>
+            <samples>720</samples>
+            <resolution>1</resolution>
+            <min_angle>0</min_angle>
+            <max_angle>3.141592</max_angle>
+          </horizontal>
+        </scan>
+        <range>
+          <min>0.5</min>
+          <max>30.0</max>
+          <resolution>0.01</resolution>
+        </range>
+        <noise>
+          <type>gaussian</type>
+          <!-- Noise parameters based on published spec for Hokuyo laser
+               achieving "+-30mm" accuracy at range < 10m.  A mean of 0.0m and
+               stddev of 0.01m will put 99.7% of samples within 0.03m of the true
+               reading. -->
+          <mean>0.0</mean>
+          <stddev>0.01</stddev>
+        </noise>
+      </ray>
+      <plugin name="gazebo_ros_fr_lidar" filename="libgazebo_ros_laser.so">
+        <topicName>sick_lidar_fr/scan</topicName>
+        <frameName>sick_lidar_fr_link</frameName>
+      </plugin>
+    </sensor>
+    </gazebo>
+    <gazebo reference="sick_lidar_rl_link">
+    <sensor type="ray" name="sick_lidar_rl">
+      <pose>0 0 0 0 0 0</pose>
+      <visualize>true</visualize>
+      <update_rate>40</update_rate>
+      <ray>
+        <scan>
+          <horizontal>
+            <samples>720</samples>
+            <resolution>1</resolution>
+            <min_angle>0</min_angle>
+            <max_angle>3.141592</max_angle>
+          </horizontal>
+        </scan>
+        <range>
+          <min>0.5</min>
+          <max>30.0</max>
+          <resolution>0.01</resolution>
+        </range>
+        <noise>
+          <type>gaussian</type>
+          <!-- Noise parameters based on published spec for Hokuyo laser
+               achieving "+-30mm" accuracy at range < 10m.  A mean of 0.0m and
+               stddev of 0.01m will put 99.7% of samples within 0.03m of the true
+               reading. -->
+          <mean>0.0</mean>
+          <stddev>0.01</stddev>
+        </noise>
+      </ray>
+      <plugin name="gazebo_ros_rl_lidar" filename="libgazebo_ros_laser.so">
+        <topicName>sick_lidar_rl/scan</topicName>
+        <frameName>sick_lidar_rl_link</frameName>
+      </plugin>
+    </sensor>
+    </gazebo>
+    <gazebo reference="sick_lidar_rr_link">
+    <sensor type="ray" name="sick_lidar_rr">
+      <pose>0 0 0 0 0 0</pose>
+      <visualize>true</visualize>
+      <update_rate>40</update_rate>
+      <ray>
+        <scan>
+          <horizontal>
+            <samples>720</samples>
+            <resolution>1</resolution>
+            <min_angle>0</min_angle>
+            <max_angle>3.141592</max_angle>
+          </horizontal>
+        </scan>
+        <range>
+          <min>0.5</min>
+          <max>30.0</max>
+          <resolution>0.01</resolution>
+        </range>
+        <noise>
+          <type>gaussian</type>
+          <!-- Noise parameters based on published spec for Hokuyo laser
+               achieving "+-30mm" accuracy at range < 10m.  A mean of 0.0m and
+               stddev of 0.01m will put 99.7% of samples within 0.03m of the true
+               reading. -->
+          <mean>0.0</mean>
+          <stddev>0.01</stddev>
+        </noise>
+      </ray>
+      <plugin name="gazebo_ros_rr_lidar" filename="libgazebo_ros_laser.so">
+        <topicName>sick_lidar_rr/scan</topicName>
+        <frameName>sick_lidar_rr_link</frameName>
+      </plugin>
+    </sensor>
+    </gazebo>
 </robot>

Commit message: colors and changed mesh

File: catkin_ws/src/4ws_robot/urdf/four_wheel_robot.xacro (robot description, xacro)
@@ -443,6 +443,7 @@
       <origin xyz="0 0 0" rpy="0 0 0"/>
       <geometry>
-        <mesh filename="package://4ws_robot/meshes/sick_lidar.obj"/>
-      </geometry>
+        <cylinder length="0.1" radius="0.03"/>
+      </geometry>
+         <material name="red"/>
     </visual>
     <inertial>
@@ -468,6 +469,7 @@
       <origin xyz="0 0 0" rpy="0 0 0"/>
       <geometry>
-        <mesh filename="package://4ws_robot/meshes/sick_lidar.obj"/>
-      </geometry>
+       <cylinder length="0.1" radius="0.03"/>
+      </geometry>
+        <material name="red"/>
     </visual>
     <inertial>
@@ -493,6 +495,7 @@
       <origin xyz="0 0 0" rpy="0 0 0"/>
       <geometry>
-        <mesh filename="package://4ws_robot/meshes/sick_lidar.obj"/>
-      </geometry>
+        <cylinder length="0.1" radius="0.03"/>
+      </geometry>
+        <material name="red"/>
     </visual>
     <inertial>
@@ -518,6 +521,7 @@
       <origin xyz="0 0 0" rpy="0 0 0"/>
       <geometry>
-        <mesh filename="package://4ws_robot/meshes/sick_lidar.obj"/>
-      </geometry>
+        <cylinder length="0.1" radius="0.03"/>
+      </geometry>
+        <material name="red"/>
     </visual>
     <inertial>
@@ -617,5 +621,5 @@
     <sensor type="ray" name="sick_lidar_fl">
       <pose>0 0 0 0 0 0</pose>
-      <visualize>true</visualize>
+      <visualize>false</visualize>
       <update_rate>40</update_rate>
       <ray>
@@ -635,8 +639,4 @@
         <noise>
           <type>gaussian</type>
-          <!-- Noise parameters based on published spec for Hokuyo laser
-               achieving "+-30mm" accuracy at range < 10m.  A mean of 0.0m and
-               stddev of 0.01m will put 99.7% of samples within 0.03m of the true
-               reading. -->
           <mean>0.0</mean>
           <stddev>0.01</stddev>
@@ -652,5 +652,5 @@
     <sensor type="ray" name="sick_lidar_fr">
       <pose>0 0 0 0 0 0</pose>
-      <visualize>true</visualize>
+      <visualize>false</visualize>
       <update_rate>40</update_rate>
       <ray>
@@ -670,8 +670,4 @@
         <noise>
           <type>gaussian</type>
-          <!-- Noise parameters based on published spec for Hokuyo laser
-               achieving "+-30mm" accuracy at range < 10m.  A mean of 0.0m and
-               stddev of 0.01m will put 99.7% of samples within 0.03m of the true
-               reading. -->
           <mean>0.0</mean>
           <stddev>0.01</stddev>
@@ -687,5 +683,5 @@
     <sensor type="ray" name="sick_lidar_rl">
       <pose>0 0 0 0 0 0</pose>
-      <visualize>true</visualize>
+      <visualize>false</visualize>
       <update_rate>40</update_rate>
       <ray>
@@ -705,8 +701,4 @@
         <noise>
           <type>gaussian</type>
-          <!-- Noise parameters based on published spec for Hokuyo laser
-               achieving "+-30mm" accuracy at range < 10m.  A mean of 0.0m and
-               stddev of 0.01m will put 99.7% of samples within 0.03m of the true
-               reading. -->
           <mean>0.0</mean>
           <stddev>0.01</stddev>
@@ -722,5 +714,5 @@
     <sensor type="ray" name="sick_lidar_rr">
       <pose>0 0 0 0 0 0</pose>
-      <visualize>true</visualize>
+      <visualize>false</visualize>
       <update_rate>40</update_rate>
       <ray>
@@ -740,8 +732,4 @@
         <noise>
           <type>gaussian</type>
-          <!-- Noise parameters based on published spec for Hokuyo laser
-               achieving "+-30mm" accuracy at range < 10m.  A mean of 0.0m and
-               stddev of 0.01m will put 99.7% of samples within 0.03m of the true
-               reading. -->
           <mean>0.0</mean>
           <stddev>0.01</stddev>
@@ -754,3 +742,19 @@
     </sensor>
     </gazebo>
+<!-- COLORS -->
+   <material name="Red"> -->
+    <color rgba="${255/255} ${0} ${0} 1.0"/>
+  </material>
+<gazebo reference="sick_lidar_rr_link">
+    <material>Gazebo/Red</material>
+  </gazebo>
+  <gazebo reference="sick_lidar_rl_link">
+    <material>Gazebo/Red</material>
+  </gazebo>
+  <gazebo reference="sick_lidar_fr_link">
+    <material>Gazebo/Red</material>
+  </gazebo>
+  <gazebo reference="sick_lidar_fl_link">
+    <material>Gazebo/Red</material>
+  </gazebo>
 </robot>
