Commit message: localization lidars package

File: gen0_hw/src/gen0_main/urdf/description.xacro (robot description, xacro)
@@ -421,10 +421,62 @@
         </inertial>
     </link>
-<!-- Lidars to be installed -->
+<!-- Localization Lidars -->
   <!-- <xacro:include filename="$(find 4ws_robot)/urdf/os1_64.urdf.xacro"/>
   <xacro:os1_64 parent="base" name="ouster" prefix="/os1_cloud_node" hz="10" samples="512">
     <origin xyz="0 0 3.0" rpy="0 0 0" />
   </xacro:os1_64> -->
-<!-- Lidars to be installed -->
+  <joint name="top_lidar_front_joint" type="fixed">
+    <axis xyz="0 1 0" />
+    <origin xyz="0.2 0 3.0" rpy="0 0 0"/>
+    <parent link="base_link"/>
+    <child link="top_lidar_front_link"/>
+  </joint>
+  <link name="top_lidar_front_link">
+    <collision>
+      <origin xyz="0 0 0" rpy="0 0 0"/>
+      <geometry>
+    <box size="0.1 0.1 0.1"/>
+      </geometry>
+    </collision>
+    <visual>
+      <origin xyz="0 0 0" rpy="0 0 0"/>
+      <geometry>
+        <box size="0.1 0.1 0.1"/>
+      </geometry>
+         <material name="blue"/>
+    </visual>
+    <inertial>
+      <mass value="1e-5" />
+      <origin xyz="0 0 0" rpy="0 0 0"/>
+      <inertia ixx="1e-6" ixy="0" ixz="0" iyy="1e-6" iyz="0" izz="1e-6" />
+    </inertial>
+  </link>
+  <joint name="top_lidar_rear_joint" type="fixed">
+    <axis xyz="0 1 0" />
+    <origin xyz="-0.2 0 3.0" rpy="0 0 3.14"/>
+    <parent link="base_link"/>
+    <child link="top_lidar_rear_link"/>
+  </joint>
+  <link name="top_lidar_rear_link">
+    <collision>
+      <origin xyz="0 0 0" rpy="0 0 0"/>
+      <geometry>
+    <box size="0.1 0.1 0.1"/>
+      </geometry>
+    </collision>
+    <visual>
+      <origin xyz="0 0 0" rpy="0 0 0"/>
+      <geometry>
+        <box size="0.1 0.1 0.1"/>
+      </geometry>
+         <material name="blue"/>
+    </visual>
+    <inertial>
+      <mass value="1e-5" />
+      <origin xyz="0 0 0" rpy="0 0 0"/>
+      <inertia ixx="1e-6" ixy="0" ixz="0" iyy="1e-6" iyz="0" izz="1e-6" />
+    </inertial>
+  </link>
+<!-- Navigation Lidars -->
 <joint name="sick_lidar_fl_joint" type="fixed">
     <axis xyz="0 1 0" />
@@ -535,3 +587,6 @@
     <color rgba="${255/255} ${0} ${0} 1.0"/>
   </material>
+   <material name="Blue"> -->
+    <color rgba="${0} ${0} ${255/255} 1.0"/>
+  </material>
 </robot>

Commit message: latest TEB parameters & new experiment maps

File: gen0_hw/src/gen0_main/urdf/description.xacro (robot description, xacro)
@@ -69,5 +69,5 @@
       <parent link="base_link"/>
       <child link="main_mass"/>
-      <origin xyz="0 0 0" rpy="0 0 0"/>
+      <origin xyz="0.0 0 0" rpy="0 0 0"/>
   </joint>
   <link name="main_mass" type="fixed">
