Commit message: relative directories update

File: gen0_main/urdf/description.urdf.xacro (robot description, xacro)
@@ -61,5 +61,5 @@
       <origin xyz="0 0 0" rpy="0 0 -1.57079633"/>
       <geometry>
-        <mesh filename="/home/av-lab/Documents/GitHub/ezmile_gen0/gen0_simulator/src/gen0_main/meshes/gen0_colored.dae"/>
+        <mesh filename="./meshes/gen0_colored.dae"/>
       </geometry>
     </visual>
@@ -152,5 +152,5 @@
                 <!--cylinder length="${tyre_length}" radius="${tyre_radius}"/>
                 <scale xyz="1 1 1"/-->
-                <mesh scale="1.2 1 1" filename="/home/av-lab/Documents/GitHub/ezmile_gen0/gen0_simulator/src/gen0_main/meshes/gen0_wheels.dae"/>
+                <mesh scale="1.2 1 1" filename="./meshes/gen0_wheels.dae"/>
             </geometry>
         </visual>
@@ -235,5 +235,5 @@
             <geometry>
                 <!--cylinder length="${tyre_length}" radius="${tyre_radius}"/-->
-                <mesh scale="1.2 1 1" filename="/home/av-lab/Documents/GitHub/ezmile_gen0/gen0_simulator/src/gen0_main/meshes/gen0_wheels.dae"/>
+                <mesh scale="1.2 1 1" filename="./meshes/gen0_wheels.dae"/>
             </geometry>
         </visual>
@@ -321,5 +321,5 @@
                 <!--cylinder length="${tyre_length}" radius="${tyre_radius}"/>
                 <scale xyz="1 1 1"/-->
-                <mesh scale="1.2 1 1" filename="/home/av-lab/Documents/GitHub/ezmile_gen0/gen0_simulator/src/gen0_main/meshes/gen0_wheels.dae"/>
+                <mesh scale="1.2 1 1" filename="./meshes/gen0_wheels.dae"/>
                 </geometry>
         </visual>
@@ -408,5 +408,5 @@
             <geometry>
             <!--cylinder length="${tyre_length}" radius="${tyre_radius}"/-->
-            <mesh scale="1.2 1 1" filename="/home/av-lab/Documents/GitHub/ezmile_gen0/gen0_simulator/src/gen0_main/meshes/gen0_wheels.dae"/>
+            <mesh scale="1.2 1 1" filename="./meshes/gen0_wheels.dae"/>
             </geometry>
         </visual>
